Commit message: lifter_moveit_taha

File: my_bot/description/gazebo_control.xacro (robot description, xacro)
@@ -25,3 +25,10 @@
         </plugin>
     </gazebo>
+     <gazebo>
+      <plugin filename="libgazebo_ros2_control.so" name="gazebo_ros2_control">
+        <robot_param>robot_description</robot_param>
+        <robot_param_node>robot_state_publisher</robot_param_node>
+        <parameters>$(find arduinobot_controller)/config/arduinobot_controllers.yaml</parameters>
+      </plugin>
+    </gazebo>
 </robot>

File: my_bot/description/robot.urdf.xacro (robot description, xacro)
@@ -3,4 +3,5 @@
     <xacro:include filename="robot_core.xacro"/>
     <xacro:include filename="gazebo_control.xacro"/>
+    <xacro:include filename="arduinobot_ros2_control.xacro"/>
     <xacro:include filename="lidar.xacro"/>
     <!--xacro:include filename="depth_camera.xacro"/-->

File: my_bot/description/robot_core.xacro (robot description, xacro)
@@ -134,3 +134,79 @@
         <mu2 value="0.0005"/>
     </gazebo>
+  <xacro:macro name="lifter_transmission" params="joint_name actuator_name">
+    <transmission name="${joint_name}_transmission">
+        <plugin>transmission_interface/SimpleTransmission</plugin>
+        <actuator name="${actuator_name}" role="actuator1"/>
+        <joint name="${joint_name}" role="joint1">
+            <mechanical_reduction>1.0</mechanical_reduction>
+        </joint>
+    </transmission>
+  </xacro:macro>
+  <xacro:property name="screw_diameter" value="0.008" />
+  <xacro:property name="screw_length" value="0.10" />
+  <xacro:property name="plate_radius" value="0.045" />
+    <!-- Link for the platform mid -->
+  <link name="link_platform_mid">
+    <origin xyz="0 0 0.0" rpy="0 0 0"/>
+    <visual>
+      <geometry>
+        <mesh filename="package://my_bot/meshes/Lead_screw.STL" scale="0.001 0.001 0.001" />
+      </geometry>
+      <material name="black">
+        <color rgba="0.1 0.1 0.1 1" />
+      </material>
+    </visual>
+    <collision>
+      <geometry>
+        <box size="0.02 0.02 0.10" />
+      </geometry>
+    </collision>
+    <inertial>
+      <mass value="1"/>
+      <inertia ixx="1.0" ixy="0.0" ixz="0.0"
+               iyy="1.0" iyz="0.0"
+               izz="1.0"/>
+    </inertial>
+  </link>
+  <!-- Joint connecting upper link to platform mid -->
+  <joint name="platform_joint" type="fixed">
+    <parent link="chassis" />
+    <child link="link_platform_mid" />
+    <origin xyz="0.0 0 0.02" rpy="0 0 0"/>
+  </joint>
+  <!-- Link for the lift mechanism -->
+  <link name="lift_link">
+    <visual>
+      <origin xyz="-${plate_radius/1.1} -${plate_radius/1.1}  0.0" rpy="0 0 0"/>
+      <geometry>
+        <mesh filename="package://arduinobot_description/meshes/upperstand.STL" scale="0.001 0.001 0.001" />
+      </geometry>
+      <material name="black">
+        <color rgba="0.1 0.1 0.1 1" />
+      </material>
+    </visual>
+    <collision>
+      <geometry>
+        <mesh filename="package://my_bot/meshes/upperstand.STL" scale="0.001 0.001 0.001" />
+      </geometry>
+    </collision>
+    <inertial>
+      <mass value="1"/>
+      <inertia ixx="1.0" ixy="0.0" ixz="0.0"
+               iyy="1.0" iyz="0.0"
+               izz="1.0"/>
+    </inertial>
+  </link>
+  <!-- Prismatic joint for lifting -->
+  <joint name="lift_joint" type="prismatic">
+    <origin xyz="0 0 0.03" rpy="0 0 0"/>
+    <parent link="link_platform_mid" />
+    <child link="lift_link" />
+    <axis xyz="0 0 1" rpy="0 0 0"/>
+    <limit effort="100.0" lower="-0.05" upper="0.035" velocity="1.0"/>
+    <dynamics damping="0.1" friction="0.1"/>
+    <hardwareInterface>hardware_interface/VelocityJointInterface</hardwareInterface>
+  </joint>
+ <!-- Use the lifter transmission macro for lift_joint -->
+ <lifter_transmission joint_name="lift_joint" actuator_name="lifter_motor"/>
 </robot>
