Commit message: adjust_lift_and_lidar_position

File: my_bot/description/lidar.xacro (robot description, xacro)
@@ -4,5 +4,5 @@
         <parent link="chassis"/>
         <child link="laser_frame"/>
-        <origin xyz="0.1 0 0.175" rpy="0 0 0"/>
+        <origin xyz="0.1 0 0.17" rpy="0 0 0"/>
     </joint>
     <link name="laser_frame">

File: my_bot/description/robot_core.xacro (robot description, xacro)
@@ -173,5 +173,5 @@
     <parent link="chassis" />
     <child link="link_platform_mid" />
-    <origin xyz="0.0 0 0.02" rpy="0 0 0"/>
+    <origin xyz="0.25 0 0.15" rpy="0 0 0"/>
   </joint>
   <!-- Link for the lift mechanism -->
@@ -180,5 +180,5 @@
       <origin xyz="-${plate_radius/1.1} -${plate_radius/1.1}  0.0" rpy="0 0 0"/>
       <geometry>
-        <mesh filename="package://arduinobot_description/meshes/upperstand.STL" scale="0.001 0.001 0.001" />
+        <mesh filename="package://my_bot/meshes/upperstand.STL" scale="0.001 0.001 0.001" />
       </geometry>
       <material name="black">
@@ -204,5 +204,5 @@
     <child link="lift_link" />
     <axis xyz="0 0 1" rpy="0 0 0"/>
-    <limit effort="100.0" lower="-0.05" upper="0.035" velocity="1.0"/>
+    <limit effort="100.0" lower="-0.05" upper="0.5" velocity="1.0"/>
     <dynamics damping="0.1" friction="0.1"/>
     <hardwareInterface>hardware_interface/VelocityJointInterface</hardwareInterface>
