Commit message: launch files with 2 wheels

File: my_bot/description/lift.xacro (robot description, xacro)
@@ -49,5 +49,5 @@
       <origin xyz="0 0  0.0" rpy="0 0 0"/>
       <geometry>
-        <cylinder radius="0.14" length="0.0015"/>
+        <cylinder radius="0.24" length="0.0015"/>
       </geometry>
       <material name="black">
