Commit message: return_to_bumper_bot_but_not_working

File: robitcubebot_description/urdf/imu.xacro (robot description, xacro)
@@ -12,5 +12,5 @@
       <origin xyz="0 0 0" rpy="0 0 0" />
       <geometry>
-        <mesh filename="package://robitcubebot_description/meshes/imu_link.STL" scale="0.4 1.3 0.5"/>
+        <mesh filename="package://robitcubebot_description/meshes/imu_link.STL" />
       </geometry>
       <material name="">
@@ -26,8 +26,58 @@
   </link>
   <joint name="imu_joint" type="fixed">
-    <origin xyz="0.065 0.012 0.043" rpy="0 0 0" />
-    <parent link="upper_link" />
+    <origin xyz="0 0 0.0698986241758014" rpy="0 0 0" />
+    <parent link="base_link" />
     <child link="imu_link" />
     <axis xyz="0 0 0" />
   </joint>
+  <!-- IMU -->
+  <gazebo reference="imu_link">
+    <sensor name="imu" type="imu">
+        <always_on>true</always_on>
+        <update_rate>100</update_rate>
+        <imu>
+          <angular_velocity>
+            <x>
+              <noise type="gaussian">
+                <mean>0.0</mean>
+                <stddev>2e-4</stddev>
+              </noise>
+            </x>
+            <y>
+              <noise type="gaussian">
+                <mean>0.0</mean>
+                <stddev>2e-4</stddev>
+              </noise>
+            </y>
+            <z>
+              <noise type="gaussian">
+                <mean>0.0</mean>
+                <stddev>2e-4</stddev>
+              </noise>
+            </z>
+          </angular_velocity>
+          <linear_acceleration>
+            <x>
+              <noise type="gaussian">
+                <mean>0.0</mean>
+                <stddev>1.7e-2</stddev>
+              </noise>
+            </x>
+            <y>
+              <noise type="gaussian">
+                <mean>0.0</mean>
+                <stddev>1.7e-2</stddev>
+              </noise>
+            </y>
+            <z>
+              <noise type="gaussian">
+                <mean>0.0</mean>
+                <stddev>1.7e-2</stddev>
+              </noise>
+            </z>
+          </linear_acceleration>
+        </imu>
+        <plugin name="imu" filename="libgazebo_ros_imu_sensor.so"/>
+    </sensor>
+  </gazebo>
 </robot>

File: robitcubebot_description/urdf/lift.xacro (robot description, xacro)
@@ -29,5 +29,5 @@
   </link>
   <joint name="platform_joint" type="fixed">
-    <parent link="upper_link" />
+    <parent link="base_link" />
     <child link="link_platform_mid" />
     <origin xyz="0.0 0 0.02" rpy="0. 0. 0."/>

File: robitcubebot_description/urdf/robitcubebot.urdf.xacro (robot description, xacro)
@@ -4,8 +4,42 @@
   <xacro:arg name="is_sim" default="true"/>
   <!-- Include Gazebo Parameters -->
-  <xacro:include filename="$(find robitcubebot_description)/urdf/robitcubebot_gazebo.xacro" />
+  <!--xacro:include filename="robitcubebot_gazebo.xacro" /-->
+  <!-- Move this one to ros2 control -->
+  <transmission name="wheel_right_transmission">
+    <plugin>transmission_interface/SimpleTransmission</plugin>
+    <actuator name="wheel_right_motor" role="actuator_right"/>
+    <joint name="wheel_right_joint"    role="joint_right">
+      <mechanical_reduction>1.0</mechanical_reduction>
+    </joint>
+  </transmission>
+  <transmission name="wheel_left_transmission">
+    <plugin>transmission_interface/SimpleTransmission</plugin>
+    <actuator name="wheel_left_motor" role="actuator_left"/>
+    <joint name="wheel_left_joint"    role="joint_left">
+      <mechanical_reduction>1.0</mechanical_reduction>
+    </joint>
+  </transmission>
+  <!-- Wheels -->
+  <gazebo reference="wheel_left_link">
+    <mu1>1000000000000000.0</mu1>
+    <mu2>1000000000000000.0</mu2>
+    <kp>1000000000000.0</kp>
+    <kd>10.0</kd>
+    <minDepth>0.001</minDepth>
+    <maxVel>0.1</maxVel>
+    <fdir1>1 0 0</fdir1>
+  </gazebo>
+  <gazebo reference="wheel_right_link">
+    <mu1>1000000000000000.0</mu1>
+    <mu2>1000000000000000.0</mu2>
+    <kp>1000000000000.0</kp>
+    <kd>10.0</kd>
+    <minDepth>0.001</minDepth>
+    <maxVel>0.1</maxVel>
+    <fdir1>1 0 0</fdir1>
+  </gazebo>
   <!-- Include ros2_control Plugins -->
   <xacro:include filename="common_properties.xacro" />
-  <xacro:include filename="$(find robitcubebot_description)/urdf/robitcubebot_ros2_control.xacro" />
+  <xacro:include filename="robitcubebot_ros2_control.xacro" />
   <xacro:include filename="robitcubebot_base.xacro" />
   <xacro:include filename="lidar.xacro"/>

File: robitcubebot_description/urdf/robitcubebot_base.xacro (robot description, xacro)
@@ -1,39 +1,47 @@
 <?xml version="1.0"?>
 <robot name="robitcubebot" xmlns:xacro="http://ros.org/wiki/xacro">
-  <xacro:include filename="common_properties.xacro" />
-  <link name="base_footprint"/>
-  <!-- Define robot properties -->
+  <!-- Load Simulated or Real Hardware Interfaces -->
+  <xacro:arg name="is_sim" default="true"/>
   <xacro:property name="base_length" value="0.317" />
   <xacro:property name="base_width" value="0.212" />
   <xacro:property name="base_height" value="0.0446" />
+  <xacro:property name="upper_length" value="0.317" />
+  <xacro:property name="upper_width" value="0.212" />
+  <xacro:property name="upper_height" value="0.0423" />
   <xacro:property name="wheel_radius" value="0.0325" />
-  <xacro:property name="wheel_length" value="0.025" />
+  <xacro:property name="wheel_length" value="0.028" />
+  <xacro:property name="to_wheel_center" value="0.07" />
+  <!-- Include Gazebo Parameters -->
+  <xacro:include filename="$(find robitcubebot_description)/urdf/robitcubebot_gazebo.xacro" />
+  <!-- Include ros2_control Plugins -->
+  <xacro:include filename="$(find robitcubebot_description)/urdf/robitcubebot_ros2_control.xacro" />
+  <link name="base_footprint"/>
   <link name="base_link">
-    <xacro:box_inertia m="0.6" l="${2*base_length}" w="${2*base_width}" h="${2*base_height}"
-                           xyz="0 0 ${base_height / 2.0}" rpy="0 0 0" />
+    <inertial>
+      <origin xyz="0 0 0.04" rpy="0.0 0.25 0.3" />
+      <mass value="8.2573504e-01"/>
+      <inertia ixx="2.2124416e-02" ixy="-1.2294101e-04" ixz="3.4938785e-04"
+               iyy="2.1193702e-02" iyz="-5.0120904e-05"
+               izz="2.0064271e-02" />
+    </inertial>
     <visual>
-      <origin xyz="-${base_length / 2.0} -${base_width / 2.0} 0" rpy="0 0 0" />
+      <origin xyz="0 0 0" rpy="0 0 0" />
       <geometry>
-        <mesh filename="package://robitcubebot_description/meshes/base_link.STL" scale="0.001 0.001 0.001" />
+        <mesh filename="package://robitcubebot_description/meshes/base_link.STL" />
       </geometry>
-      <material name="black">
-          <color rgba="0.1 0.1 0.1 1" />
-      </material>
     </visual>
     <collision>
-      <origin xyz="0 0 0.1" rpy="0 0 0" />
+      <origin xyz="0 0 0" rpy="0 0 0" />
       <geometry>
-        <box size="${base_length} ${base_width} ${base_height}" />
+        <mesh filename="package://robitcubebot_description/meshes/base_link.STL" />
       </geometry>
     </collision>
   </link>
-  <!-- Define joints -->
   <joint name="base_joint" type="fixed">
     <parent link="base_footprint"/>
     <child link="base_link" />
-    <origin xyz="0 0 0" rpy="0 0 0"/>
+    <origin xyz="0 0 0.033" rpy="0 0 0"/>
   </joint>
-  <!-- Wheels -->
-  <link name="front_wheel_right_link">
+  <link name="wheel_right_link">
     <inertial>
       <origin xyz="0 -0.014 0" rpy="0 0 0" />
@@ -56,12 +64,12 @@
     </collision>
   </link>
-  <joint name="front_wheel_right_joint" type="continuous">
-    <origin xyz="-${base_width / 1.8} -${base_width / 2.1} ${wheel_radius}" rpy="0 0 0" />
+  <joint name="wheel_right_joint" type="continuous">
+    <origin xyz="0 -0.0701101849418637 0" rpy="0 0 0" />
     <parent link="base_link" />
-    <child link="front_wheel_right_link" />
-    <axis xyz="0 -1 0" />
+    <child link="wheel_right_link" />
+    <axis xyz="0 1 0" />
   </joint>
   <link
-    name="front_wheel_left_link">
+    name="wheel_left_link">
     <inertial>
       <origin xyz="0 0.014 0" rpy="0 0 0" />
@@ -84,88 +92,63 @@
     </collision>
   </link>
-  <joint name="front_wheel_left_joint" type="continuous">
-    <origin xyz="-${base_width / 1.8} ${base_width / 2.1} ${wheel_radius}" rpy="0 0 0" />
+  <joint name="wheel_left_joint" type="continuous">
+    <origin xyz="0 0.0701101849418642 0" rpy="0 0 0" />
     <parent link="base_link" />
-    <child link="front_wheel_left_link" />
-    <axis xyz="0 -1 0" />
+    <child link="wheel_left_link" />
+    <axis xyz="0 1 0" />
   </joint>
-  <link name="back_wheel_right_link">
+  <link name="caster_front_link">
     <inertial>
-      <origin xyz="0 -0.014 0" rpy="0 0 0" />
-      <mass value="0.0530086090966721" />
-      <inertia ixx="1.88176298336665E-05" ixy="-4.8444933029987E-10" ixz="1.88163708851143E-08"
-               iyy="3.11510738647764E-05" iyz="-6.93560663069607E-11"
-               izz="1.8801969558182E-05" />
+      <origin xyz="3.89968128948481E-07 2.40073004698083E-07 0.00219173397061506" rpy="0 0 0" />
+      <mass value="1.44379265037903E-06" />
+      <inertia ixx="7.23075276010246E-11" ixy="-6.10956883467859E-16" ixz="2.22849693525031E-15"
+               iyy="3.8713793085917E-11"  iyz="2.93909858781952E-15"
+               izz="1.00967486676306E-10" />
     </inertial>
     <visual>
-      <origin xyz="0 0 0" rpy="1.57 0 0" />
+      <origin xyz="0 0 0" rpy="0 0 0" />
       <geometry>
-        <mesh filename="package://robitcubebot_description/meshes/wheel_right_link.STL" />
+        <mesh filename="package://robitcubebot_description/meshes/caster_front_link.STL" />
       </geometry>
     </visual>
     <collision>
-      <origin xyz="0 -0.015 0" rpy="1.57 0 0" />
+      <origin xyz="0 0 0" rpy="0 0 0" />
       <geometry>
-        <sphere radius="0.033"/>
+        <sphere radius="0.005"/>
       </geometry>
     </collision>
   </link>
-  <joint name="back_wheel_right_joint" type="continuous">
-    <origin xyz="${base_width / 1.8} -${base_width / 2.1} ${wheel_radius}" rpy="0 0 0" />
+  <joint name="caster_front_joint" type="fixed">
+    <origin xyz="0.04755 0 -0.0275" rpy="0 0 0" />
     <parent link="base_link" />
-    <child link="back_wheel_right_link" />
-    <axis xyz="0 -1 0" />
+    <child link="caster_front_link" />
+    <axis xyz="0 0 0" />
   </joint>
-  <link
-    name="back_wheel_left_link">
+  <link name="caster_rear_link">
     <inertial>
-      <origin xyz="0 0.014 0" rpy="0 0 0" />
-      <mass value="0.0530086043217644" />
-      <inertia ixx="1.8792911368909E-05"  ixy="3.31256392204584E-10" ixz="-1.14082001662767E-08"
-               iyy="3.11510738759073E-05" iyz="-3.60499245082192E-10"
-               izz="1.88266886146847E-05" />
+      <origin xyz="3.8996812895542E-07 2.40073004698083E-07 0.00219173397061509" rpy="0 0 0" />
+      <mass value="1.44379265037902E-06" />
+      <inertia ixx="7.23075276010246E-11" ixy="-6.10956872363424E-16" ixz="2.22849693527207E-15"
+               iyy="3.87137930859167E-11" iyz="2.939098587861E-15"
+               izz="1.00967486676306E-10" />
     </inertial>
     <visual>
-      <origin xyz="0 0 0" rpy="-1.57 0 0" />
+      <origin xyz="0 0 0" rpy="0 0 0" />
       <geometry>
-        <mesh filename="package://robitcubebot_description/meshes/wheel_left_link.STL" />
+        <mesh filename="package://robitcubebot_description/meshes/caster_rear_link.STL" />
       </geometry>
     </visual>
     <collision>
-      <origin xyz="0 0.015 0" rpy="-1.57 0 0" />
+      <origin xyz="0 0 0" rpy="0 0 0" />
       <geometry>
-        <sphere radius="0.033"/>
+        <sphere radius="0.005"/>
       </geometry>
     </collision>
   </link>
-  <joint name="back_wheel_left_joint" type="continuous">
-    <origin xyz="${base_width / 1.8} ${base_width / 2.1} ${wheel_radius}" rpy="0 0 0" />
+  <joint name="caster_rear_joint" type="fixed">
+    <origin xyz="-0.04755 0 -0.0275" rpy="0 0 0" />
     <parent link="base_link" />
-    <child link="back_wheel_left_link" />
-    <axis xyz="0 -1 0" />
-  </joint>
-  <link name="upper_link">
-    <xacro:box_inertia m="0.6" l="${2*base_length}" w="${2*base_width}" h="${2*base_height}"
-                           xyz="0 0 ${base_height / 2.0}" rpy="0 0 0" />
-    <visual>
-      <origin xyz="-${base_length / 1.75} -0.165 0" rpy="0 0 0" />
-      <geometry>
-        <mesh filename="package://robitcubebot_description/meshes/upper_link.STL" scale="0.001 0.001 0.001" />
-      </geometry>
-      <material name="black">
-        <color rgba="0.1 0.1 0.1 1" />
-      </material>
-    </visual>
-    <collision>
-      <origin xyz="0 0 ${base_height}" rpy="0 0 0" />
-      <geometry>
-        <box size="${base_length} ${base_width} ${base_height}" />
-      </geometry>
-    </collision>
-  </link>
-  <joint name="upper_joint" type="fixed">
-    <parent link="base_link"/>
-    <child link="upper_link" />
-    <origin xyz="0 0 ${base_height}" rpy="0 0 0"/>
+    <child link="caster_rear_link" />
+    <axis xyz="0 0 0" />
   </joint>
 </robot>

File: robitcubebot_description/urdf/robitcubebot_gazebo.xacro (robot description, xacro)
@@ -2,34 +2,20 @@
 <robot name="robitcubebot" xmlns:xacro="http://ros.org/wiki/xacro">
   <!-- Move this one to ros2 control -->
-  <transmission name="front_right_wheel_transmission">
+  <transmission name="wheel_right_transmission">
     <plugin>transmission_interface/SimpleTransmission</plugin>
-    <actuator name="front_wheel_right_motor" role="front_actuator_right"/>
-    <joint name="front_wheel_right_joint"    role="front_joint_right">
+    <actuator name="wheel_right_motor" role="actuator_right"/>
+    <joint name="wheel_right_joint"    role="joint_right">
       <mechanical_reduction>1.0</mechanical_reduction>
     </joint>
   </transmission>
-  <transmission name="front_left_wheel_transmission">
+  <transmission name="wheel_left_transmission">
     <plugin>transmission_interface/SimpleTransmission</plugin>
-    <actuator name="front_wheel_left_motor" role="front_actuator_left"/>
-    <joint name="front_wheel_left_joint"    role="front_joint_left">
-      <mechanical_reduction>1.0</mechanical_reduction>
-    </joint>
-  </transmission>
-  <transmission name="back_right_wheel_transmission">
-    <plugin>transmission_interface/SimpleTransmission</plugin>
-    <actuator name="back_wheel_right_motor" role="back_actuator_right"/>
-    <joint name="back_wheel_right_joint"    role="back_joint_right">
-      <mechanical_reduction>1.0</mechanical_reduction>
-    </joint>
-  </transmission>
-  <transmission name="back_left_wheel_transmission">
-    <plugin>transmission_interface/SimpleTransmission</plugin>
-    <actuator name="back_wheel_left_motor" role="back_actuator_left"/>
-    <joint name="back_wheel_left_joint"    role="back_joint_left">
+    <actuator name="wheel_left_motor" role="actuator_left"/>
+    <joint name="wheel_left_joint"    role="joint_left">
       <mechanical_reduction>1.0</mechanical_reduction>
     </joint>
   </transmission>
   <!-- Wheels -->
-  <gazebo reference="front_wheel_left_link">
+  <gazebo reference="wheel_left_link">
     <mu1>1000000000000000.0</mu1>
     <mu2>1000000000000000.0</mu2>
@@ -40,5 +26,5 @@
     <fdir1>1 0 0</fdir1>
   </gazebo>
-  <gazebo reference="front_wheel_right_link">
+  <gazebo reference="wheel_right_link">
     <mu1>1000000000000000.0</mu1>
     <mu2>1000000000000000.0</mu2>
@@ -49,20 +35,4 @@
     <fdir1>1 0 0</fdir1>
   </gazebo>
-  <gazebo reference="back_wheel_left_link">
-    <mu1>0.1</mu1>
-    <mu2>0.1</mu2>
-    <kp>1000000.0</kp>
-    <kd>100.0</kd>
-    <minDepth>0.001</minDepth>
-    <maxVel>1.0</maxVel>
-  </gazebo>
-  <gazebo reference="back_wheel_right_link">
-    <mu1>0.1</mu1>
-    <mu2>0.1</mu2>
-    <kp>1000000.0</kp>
-    <kd>100.0</kd>
-    <minDepth>0.001</minDepth>
-    <maxVel>1.0</maxVel>
-  </gazebo>
   <!-- ROS 2 Control -->
   <gazebo>
@@ -70,56 +40,6 @@
       <robot_param>robot_description</robot_param>
       <robot_param_node>robot_state_publisher</robot_param_node>
-      <parameters>$(find robitcubebot_controller)/config/robitcubebot_controllers.yaml</parameters>
+      <parameters>$(find bumperbot_controller)/config/bumperbot_controllers.yaml</parameters>
     </plugin>
   </gazebo>
-  <!-- IMU -->
-  <gazebo reference="imu_link">
-    <sensor name="imu" type="imu">
-        <always_on>true</always_on>
-        <update_rate>100</update_rate>
-        <imu>
-          <angular_velocity>
-            <x>
-              <noise type="gaussian">
-                <mean>0.0</mean>
-                <stddev>2e-4</stddev>
-              </noise>
-            </x>
-            <y>
-              <noise type="gaussian">
-                <mean>0.0</mean>
-                <stddev>2e-4</stddev>
-              </noise>
-            </y>
-            <z>
-              <noise type="gaussian">
-                <mean>0.0</mean>
-                <stddev>2e-4</stddev>
-              </noise>
-            </z>
-          </angular_velocity>
-          <linear_acceleration>
-            <x>
-              <noise type="gaussian">
-                <mean>0.0</mean>
-                <stddev>1.7e-2</stddev>
-              </noise>
-            </x>
-            <y>
-              <noise type="gaussian">
-                <mean>0.0</mean>
-                <stddev>1.7e-2</stddev>
-              </noise>
-            </y>
-            <z>
-              <noise type="gaussian">
-                <mean>0.0</mean>
-                <stddev>1.7e-2</stddev>
-              </noise>
-            </z>
-          </linear_acceleration>
-        </imu>
-        <plugin name="imu" filename="libgazebo_ros_imu_sensor.so"/>
-    </sensor>
-  </gazebo>
 </robot>

File: robitcubebot_description/urdf/robitcubebot_ros2_control.xacro (robot description, xacro)
@@ -12,9 +12,9 @@
             <hardware>
                 <plugin>robitcubebot_firmware/robitcubebotInterface</plugin>
-                <param name="port">/dev/ttyACM0</param>
+                <param name="port">/dev/ttyUSB0</param>
             </hardware>
         </xacro:unless>
         <!-- ros2_control Common Interfaces -->
-        <joint name="front_wheel_right_joint">
+        <joint name="wheel_right_joint">
             <command_interface name="velocity">
               <param name="min">-1</param>
@@ -24,21 +24,5 @@
             <state_interface name="velocity" />
         </joint>
-        <joint name="front_wheel_left_joint">
-            <command_interface name="velocity">
-              <param name="min">-1</param>
-              <param name="max">1</param>
-            </command_interface>
-            <state_interface name="position" />
-            <state_interface name="velocity" />
-        </joint>
-        <joint name="back_wheel_right_joint">
-            <command_interface name="velocity">
-              <param name="min">-1</param>
-              <param name="max">1</param>
-            </command_interface>
-            <state_interface name="position" />
-            <state_interface name="velocity" />
-        </joint>
-        <joint name="back_wheel_left_joint">
+        <joint name="wheel_left_joint">
             <command_interface name="velocity">
               <param name="min">-1</param>
