Commit message: STLS

File: robitcubebot_description/urdf/imu.xacro (robot description, xacro)
@@ -31,3 +31,53 @@
     <axis xyz="0 0 0" />
   </joint>
+    <!-- IMU -->
+  <gazebo reference="imu_link">
+    <sensor name="imu" type="imu">
+        <always_on>true</always_on>
+        <update_rate>100</update_rate>
+        <imu>
+          <angular_velocity>
+            <x>
+              <noise type="gaussian">
+                <mean>0.0</mean>
+                <stddev>2e-4</stddev>
+              </noise>
+            </x>
+            <y>
+              <noise type="gaussian">
+                <mean>0.0</mean>
+                <stddev>2e-4</stddev>
+              </noise>
+            </y>
+            <z>
+              <noise type="gaussian">
+                <mean>0.0</mean>
+                <stddev>2e-4</stddev>
+              </noise>
+            </z>
+          </angular_velocity>
+          <linear_acceleration>
+            <x>
+              <noise type="gaussian">
+                <mean>0.0</mean>
+                <stddev>1.7e-2</stddev>
+              </noise>
+            </x>
+            <y>
+              <noise type="gaussian">
+                <mean>0.0</mean>
+                <stddev>1.7e-2</stddev>
+              </noise>
+            </y>
+            <z>
+              <noise type="gaussian">
+                <mean>0.0</mean>
+                <stddev>1.7e-2</stddev>
+              </noise>
+            </z>
+          </linear_acceleration>
+        </imu>
+        <plugin name="imu" filename="libgazebo_ros_imu_sensor.so"/>
+    </sensor>
+  </gazebo>
 </robot>

File: robitcubebot_description/urdf/robitcubebot.urdf.xacro (robot description, xacro)
@@ -4,11 +4,11 @@
   <xacro:arg name="is_sim" default="true"/>
   <!-- Include Gazebo Parameters -->
-  <xacro:include filename="$(find robitcubebot_description)/urdf/robitcubebot_gazebo.xacro" />
+  <!--xacro:include filename="$(find robitcubebot_description)/urdf/robitcubebot_gazebo.xacro" /-->
   <!-- Include ros2_control Plugins -->
   <xacro:include filename="common_properties.xacro" />
-  <xacro:include filename="$(find robitcubebot_description)/urdf/robitcubebot_ros2_control.xacro" />
+  <!--xacro:include filename="$(find robitcubebot_description)/urdf/robitcubebot_ros2_control.xacro" /-->
   <xacro:include filename="robitcubebot_base.xacro" />
-  <xacro:include filename="lidar.xacro"/>
-  <xacro:include filename="lift.xacro" />
-  <xacro:include filename="imu.xacro" />
+  <!--xacro:include filename="lidar.xacro"/-->
+  <!--xacro:include filename="lift.xacro" /-->
+  <!--xacro:include filename="imu.xacro" /-->
 </robot>

File: robitcubebot_description/urdf/robitcubebot_gazebo.xacro (robot description, xacro)
@@ -2,32 +2,4 @@
 <robot name="robitcubebot" xmlns:xacro="http://ros.org/wiki/xacro">
   <!-- Move this one to ros2 control -->
-  <transmission name="front_right_wheel_transmission">
-    <plugin>transmission_interface/SimpleTransmission</plugin>
-    <actuator name="front_wheel_right_motor" role="front_actuator_right"/>
-    <joint name="front_wheel_right_joint"    role="front_joint_right">
-      <mechanical_reduction>1.0</mechanical_reduction>
-    </joint>
-  </transmission>
-  <transmission name="front_left_wheel_transmission">
-    <plugin>transmission_interface/SimpleTransmission</plugin>
-    <actuator name="front_wheel_left_motor" role="front_actuator_left"/>
-    <joint name="front_wheel_left_joint"    role="front_joint_left">
-      <mechanical_reduction>1.0</mechanical_reduction>
-    </joint>
-  </transmission>
-  <transmission name="back_right_wheel_transmission">
-    <plugin>transmission_interface/SimpleTransmission</plugin>
-    <actuator name="back_wheel_right_motor" role="back_actuator_right"/>
-    <joint name="back_wheel_right_joint"    role="back_joint_right">
-      <mechanical_reduction>1.0</mechanical_reduction>
-    </joint>
-  </transmission>
-  <transmission name="back_left_wheel_transmission">
-    <plugin>transmission_interface/SimpleTransmission</plugin>
-    <actuator name="back_wheel_left_motor" role="back_actuator_left"/>
-    <joint name="back_wheel_left_joint"    role="back_joint_left">
-      <mechanical_reduction>1.0</mechanical_reduction>
-    </joint>
-  </transmission>
   <!-- Wheels -->
   <gazebo reference="front_wheel_left_link">
@@ -50,76 +22,20 @@
   </gazebo>
   <gazebo reference="back_wheel_left_link">
-    <mu1>0.1</mu1>
-    <mu2>0.1</mu2>
-    <kp>1000000.0</kp>
-    <kd>100.0</kd>
+    <mu1>1000000000000000.0</mu1>
+    <mu2>1000000000000000.0</mu2>
+    <kp>1000000000000.0</kp>
+    <kd>10.0</kd>
     <minDepth>0.001</minDepth>
-    <maxVel>1.0</maxVel>
+    <maxVel>0.1</maxVel>
+    <fdir1>1 0 0</fdir1>
   </gazebo>
   <gazebo reference="back_wheel_right_link">
-    <mu1>0.1</mu1>
-    <mu2>0.1</mu2>
-    <kp>1000000.0</kp>
-    <kd>100.0</kd>
+    <mu1>1000000000000000.0</mu1>
+    <mu2>1000000000000000.0</mu2>
+    <kp>1000000000000.0</kp>
+    <kd>10.0</kd>
     <minDepth>0.001</minDepth>
-    <maxVel>1.0</maxVel>
-  </gazebo>
-  <!-- ROS 2 Control -->
-  <gazebo>
-    <plugin filename="libgazebo_ros2_control.so" name="gazebo_ros2_control">
-      <robot_param>robot_description</robot_param>
-      <robot_param_node>robot_state_publisher</robot_param_node>
-      <parameters>$(find robitcubebot_controller)/config/robitcubebot_controllers.yaml</parameters>
-    </plugin>
-  </gazebo>
-  <!-- IMU -->
-  <gazebo reference="imu_link">
-    <sensor name="imu" type="imu">
-        <always_on>true</always_on>
-        <update_rate>100</update_rate>
-        <imu>
-          <angular_velocity>
-            <x>
-              <noise type="gaussian">
-                <mean>0.0</mean>
-                <stddev>2e-4</stddev>
-              </noise>
-            </x>
-            <y>
-              <noise type="gaussian">
-                <mean>0.0</mean>
-                <stddev>2e-4</stddev>
-              </noise>
-            </y>
-            <z>
-              <noise type="gaussian">
-                <mean>0.0</mean>
-                <stddev>2e-4</stddev>
-              </noise>
-            </z>
-          </angular_velocity>
-          <linear_acceleration>
-            <x>
-              <noise type="gaussian">
-                <mean>0.0</mean>
-                <stddev>1.7e-2</stddev>
-              </noise>
-            </x>
-            <y>
-              <noise type="gaussian">
-                <mean>0.0</mean>
-                <stddev>1.7e-2</stddev>
-              </noise>
-            </y>
-            <z>
-              <noise type="gaussian">
-                <mean>0.0</mean>
-                <stddev>1.7e-2</stddev>
-              </noise>
-            </z>
-          </linear_acceleration>
-        </imu>
-        <plugin name="imu" filename="libgazebo_ros_imu_sensor.so"/>
-    </sensor>
+    <maxVel>0.1</maxVel>
+    <fdir1>1 0 0</fdir1>
   </gazebo>
 </robot>

File: robitcubebot_description/urdf/robitcubebot_ros2_control.xacro (robot description, xacro)
@@ -56,3 +56,39 @@
         </joint>
     </ros2_control>
+    <transmission name="front_right_wheel_transmission">
+        <plugin>transmission_interface/SimpleTransmission</plugin>
+        <actuator name="front_wheel_right_motor" role="front_actuator_right"/>
+        <joint name="front_wheel_right_joint"    role="front_joint_right">
+        <mechanical_reduction>1.0</mechanical_reduction>
+        </joint>
+    </transmission>
+    <transmission name="front_left_wheel_transmission">
+        <plugin>transmission_interface/SimpleTransmission</plugin>
+        <actuator name="front_wheel_left_motor" role="front_actuator_left"/>
+        <joint name="front_wheel_left_joint"    role="front_joint_left">
+        <mechanical_reduction>1.0</mechanical_reduction>
+        </joint>
+    </transmission>
+    <transmission name="back_right_wheel_transmission">
+        <plugin>transmission_interface/SimpleTransmission</plugin>
+        <actuator name="back_wheel_right_motor" role="back_actuator_right"/>
+        <joint name="back_wheel_right_joint"    role="back_joint_right">
+        <mechanical_reduction>1.0</mechanical_reduction>
+        </joint>
+    </transmission>
+    <transmission name="back_left_wheel_transmission">
+        <plugin>transmission_interface/SimpleTransmission</plugin>
+        <actuator name="back_wheel_left_motor" role="back_actuator_left"/>
+        <joint name="back_wheel_left_joint"    role="back_joint_left">
+        <mechanical_reduction>1.0</mechanical_reduction>
+        </joint>
+    </transmission>
+      <!-- ROS 2 Control -->
+    <gazebo>
+        <plugin filename="libgazebo_ros2_control.so" name="gazebo_ros2_control">
+        <robot_param>robot_description</robot_param>
+        <robot_param_node>robot_state_publisher</robot_param_node>
+        <parameters>$(find robitcubebot_controller)/config/robitcubebot_controllers.yaml</parameters>
+        </plugin>
+    </gazebo>
 </robot>
