Commit message: lidar_plugin_updated

File: robitcubebot_description/urdf/lidar.xacro (robot description, xacro)
@@ -2,5 +2,5 @@
 <robot xmlns:xacro="http://www.ros.org/wiki/xacro" >
     <joint name="laser_joint" type="fixed">
-        <parent link="upper_link"/>
+        <parent link="base_link"/>
         <child link="laser_frame"/>
         <origin xyz="${base_length /2.5} 0.005 0.06" rpy="0 0 0"/>

Commit message: updates_in_controller_not_accurate

File: robitcubebot_description/urdf/lidar.xacro (robot description, xacro)
@@ -4,5 +4,5 @@
         <parent link="base_link"/>
         <child link="laser_frame"/>
-        <origin xyz="${base_length /2.5} 0.005 0.06" rpy="0 0 0"/>
+        <origin xyz="0 -0.005 0.12" rpy="0 0 0"/>
     </joint>
     <link name="laser_frame">

Commit message: diff drive

File: robitcubebot_description/urdf/lidar.xacro (robot description, xacro)
@@ -8,4 +8,5 @@
     <link name="laser_frame">
         <visual>
+            <origin xyz="0 0 0" rpy="0 0 0"/>
             <geometry>
                 <cylinder radius="0.034" length="0.03"/>

File: robitcubebot_description/urdf/robitcubebot.urdf.xacro (robot description, xacro)
@@ -7,5 +7,5 @@
   <!-- Include ros2_control Plugins -->
   <xacro:include filename="common_properties.xacro" />
-  <xacro:include filename="$(find robitcubebot_description)/urdf/robitcubebot_ros2_control.xacro" />
+  <!--xacro:include filename="$(find robitcubebot_description)/urdf/robitcubebot_ros2_control.xacro" /-->
   <xacro:include filename="robitcubebot_base.xacro" />
   <xacro:include filename="lidar.xacro"/>

File: robitcubebot_description/urdf/robitcubebot_base.xacro (robot description, xacro)
@@ -2,6 +2,5 @@
 <robot name="robitcubebot" xmlns:xacro="http://ros.org/wiki/xacro">
   <xacro:include filename="common_properties.xacro" />
-  <link name="base_footprint"/>
-  <!-- Define robot properties -->
+    <!-- Define robot properties -->
   <xacro:property name="base_length" value="0.317" />
   <xacro:property name="base_width" value="0.212" />
@@ -9,4 +8,11 @@
   <xacro:property name="wheel_radius" value="0.0325" />
   <xacro:property name="wheel_length" value="0.025" />
+  <link name="base_footprint"/>
+   <!-- Define joints -->
+  <joint name="base_joint" type="fixed">
+    <parent link="base_footprint"/>
+    <child link="base_link" />
+    <origin xyz="0 0 0.010" rpy="0 0 0"/>
+  </joint>
   <link name="base_link">
     <xacro:box_inertia m="0.6" l="${2*base_length}" w="${2*base_width}" h="${2*base_height}"
@@ -28,11 +34,11 @@
     </collision>
   </link>
-  <!-- Define joints -->
-  <joint name="base_joint" type="fixed">
-    <parent link="base_footprint"/>
-    <child link="base_link" />
-    <origin xyz="0 0 0" rpy="0 0 0"/>
+  <!-- Wheels -->
+   <joint name="back_wheel_left_joint" type="continuous">
+    <origin xyz="-${base_width / 1.8} -${base_width / 2} ${wheel_radius}" rpy="0 0 0" />
+    <parent link="base_link" />
+    <child link="back_wheel_left_link" />
+    <axis xyz="0 1 0" />
   </joint>
-  <!-- Wheels -->
   <link name="back_wheel_left_link">
     <inertial>
@@ -56,8 +62,8 @@
     </collision>
   </link>
-  <joint name="back_wheel_left_joint" type="continuous">
-    <origin xyz="-${base_width / 1.8} -${base_width / 2} ${wheel_radius}" rpy="0 0 0" />
+  <joint name="back_wheel_right_joint" type="continuous">
+    <origin xyz="-${base_width / 1.8} ${base_width / 2.1} ${wheel_radius}" rpy="0 0 0" />
     <parent link="base_link" />
-    <child link="back_wheel_left_link" />
+    <child link="back_wheel_right_link" />
     <axis xyz="0 1 0" />
   </joint>
@@ -84,8 +90,8 @@
     </collision>
   </link>
-  <joint name="back_wheel_right_joint" type="continuous">
-    <origin xyz="-${base_width / 1.8} ${base_width / 2.1} ${wheel_radius}" rpy="0 0 0" />
+  <joint name="front_wheel_left_joint" type="continuous">
+    <origin xyz="${base_width / 1.8} -${base_width / 2} ${wheel_radius}" rpy="0 0 0" />
     <parent link="base_link" />
-    <child link="back_wheel_right_link" />
+    <child link="front_wheel_left_link" />
     <axis xyz="0 1 0" />
   </joint>
@@ -111,8 +117,8 @@
     </collision>
   </link>
-  <joint name="front_wheel_left_joint" type="continuous">
-    <origin xyz="${base_width / 1.8} -${base_width / 2} ${wheel_radius}" rpy="0 0 0" />
+  <joint name="front_wheel_right_joint" type="continuous">
+    <origin xyz="${base_width / 1.8} ${base_width / 2.1} ${wheel_radius}" rpy="0 0 0" />
     <parent link="base_link" />
-    <child link="front_wheel_left_link" />
+    <child link="front_wheel_right_link" />
     <axis xyz="0 1 0" />
   </joint>
@@ -139,10 +145,4 @@
     </collision>
   </link>
-  <joint name="front_wheel_right_joint" type="continuous">
-    <origin xyz="${base_width / 1.8} ${base_width / 2.1} ${wheel_radius}" rpy="0 0 0" />
-    <parent link="base_link" />
-    <child link="front_wheel_right_link" />
-    <axis xyz="0 1 0" />
-  </joint>
   <link name="upper_link">
     <xacro:box_inertia m="0.6" l="${2*base_length}" w="${2*base_width}" h="${2*base_height}"

File: robitcubebot_description/urdf/robitcubebot_gazebo.xacro (robot description, xacro)
@@ -1,33 +1,4 @@
 <?xml version="1.0"?>
 <robot name="robitcubebot" xmlns:xacro="http://ros.org/wiki/xacro">
-  <!-- Move this one to ros2 control -->
-  <transmission name="front_right_wheel_transmission">
-    <plugin>transmission_interface/SimpleTransmission</plugin>
-    <actuator name="front_wheel_right_motor" role="front_actuator_right"/>
-    <joint name="front_wheel_right_joint"    role="front_joint_right">
-      <mechanical_reduction>1.0</mechanical_reduction>
-    </joint>
-  </transmission>
-  <transmission name="front_left_wheel_transmission">
-    <plugin>transmission_interface/SimpleTransmission</plugin>
-    <actuator name="front_wheel_left_motor" role="front_actuator_left"/>
-    <joint name="front_wheel_left_joint"    role="front_joint_left">
-      <mechanical_reduction>1.0</mechanical_reduction>
-    </joint>
-  </transmission>
-  <transmission name="back_right_wheel_transmission">
-    <plugin>transmission_interface/SimpleTransmission</plugin>
-    <actuator name="back_wheel_right_motor" role="back_actuator_right"/>
-    <joint name="back_wheel_right_joint"    role="back_joint_right">
-      <mechanical_reduction>1.0</mechanical_reduction>
-    </joint>
-  </transmission>
-  <transmission name="back_left_wheel_transmission">
-    <plugin>transmission_interface/SimpleTransmission</plugin>
-    <actuator name="back_wheel_left_motor" role="back_actuator_left"/>
-    <joint name="back_wheel_left_joint"    role="back_joint_left">
-      <mechanical_reduction>1.0</mechanical_reduction>
-    </joint>
-  </transmission>
   <!-- Wheels -->
   <gazebo reference="front_wheel_left_link">
@@ -38,5 +9,4 @@
     <minDepth>0.001</minDepth>
     <maxVel>0.1</maxVel>
-    <fdir1>1 0 0</fdir1>
   </gazebo>
   <gazebo reference="front_wheel_right_link">
@@ -47,28 +17,56 @@
     <minDepth>0.001</minDepth>
     <maxVel>0.1</maxVel>
-    <fdir1>1 0 0</fdir1>
   </gazebo>
   <gazebo reference="back_wheel_left_link">
-    <mu1>0.1</mu1>
-    <mu2>0.1</mu2>
-    <kp>1000000.0</kp>
-    <kd>100.0</kd>
+    <mu1>1000000000000000.0</mu1>
+    <mu2>1000000000000000.0</mu2>
+    <kp>1000000000000.0</kp>
+    <kd>10.0</kd>
     <minDepth>0.001</minDepth>
-    <maxVel>1.0</maxVel>
+    <maxVel>0.1</maxVel>
   </gazebo>
   <gazebo reference="back_wheel_right_link">
-    <mu1>0.1</mu1>
-    <mu2>0.1</mu2>
-    <kp>1000000.0</kp>
-    <kd>100.0</kd>
+    <mu1>1000000000000000.0</mu1>
+    <mu2>1000000000000000.0</mu2>
+    <kp>1000000000000.0</kp>
+    <kd>10.0</kd>
     <minDepth>0.001</minDepth>
-    <maxVel>1.0</maxVel>
+    <maxVel>0.1</maxVel>
   </gazebo>
   <!-- ROS 2 Control -->
-  <gazebo>
+  <!--gazebo>
     <plugin filename="libgazebo_ros2_control.so" name="gazebo_ros2_control">
       <robot_param>robot_description</robot_param>
       <robot_param_node>robot_state_publisher</robot_param_node>
       <parameters>$(find robitcubebot_controller)/config/robitcubebot_controllers.yaml</parameters>
+    </plugin>
+  </gazebo-->
+<gazebo>
+    <plugin name="wheel_drive_controller" filename="libgazebo_ros_diff_drive.so">
+        <!-- wheels -->
+        <num_wheel_pairs>2</num_wheel_pairs>
+        <left_joint>front_wheel_right_joint</left_joint>
+        <left_joint>back_wheel_right_joint</left_joint>
+        <right_joint>front_wheel_left_joint</right_joint>
+        <right_joint>back_wheel_left_joint</right_joint>
+        <!-- kinematics -->
+        <wheel_separation>0.4</wheel_separation>
+        <wheel_diameter>0.065</wheel_diameter>
+        <!-- Limits -->
+        <max_wheel_torque>200.0</max_wheel_torque>
+        <max_wheel_acceleration>10.0</max_wheel_acceleration>
+        <!-- Output -->
+        <odometry_frame>odom</odometry_frame>
+        <robot_base_frame>base_footprint</robot_base_frame>
+        <!-- topic & re remappings -->
+        <!-- ros>
+            <namespace>/</namespace>
+            <argument>/cmd_vel:=cmd_vel</argument>
+            <argument>/odom:=odom</argument>
+        </ros -->
+        <publish_odom>true</publish_odom>
+        <publish_odom_tf>true</publish_odom_tf>
+        <publish_wheel_tf>true</publish_wheel_tf>
+        <update_rate>30.0</update_rate>
     </plugin>
   </gazebo>

File: robitcubebot_description/urdf/robitcubebot_ros2_control.xacro (robot description, xacro)
@@ -1,4 +1,33 @@
 <?xml version="1.0"?>
 <robot xmlns:xacro="http://www.ros.org/wiki/xacro" name="robitcubebot">
+     <!-- Move this one to ros2 control -->
+    <transmission name="front_right_wheel_transmission">
+        <plugin>transmission_interface/SimpleTransmission</plugin>
+        <actuator name="front_wheel_right_motor" role="front_actuator_right"/>
+        <joint name="front_wheel_right_joint"    role="front_joint_right">
+        <mechanical_reduction>1.0</mechanical_reduction>
+        </joint>
+    </transmission>
+    <transmission name="front_left_wheel_transmission">
+        <plugin>transmission_interface/SimpleTransmission</plugin>
+        <actuator name="front_wheel_left_motor" role="front_actuator_left"/>
+        <joint name="front_wheel_left_joint"    role="front_joint_left">
+        <mechanical_reduction>1.0</mechanical_reduction>
+        </joint>
+    </transmission>
+    <transmission name="back_right_wheel_transmission">
+        <plugin>transmission_interface/SimpleTransmission</plugin>
+        <actuator name="back_wheel_right_motor" role="back_actuator_right"/>
+        <joint name="back_wheel_right_joint"    role="back_joint_right">
+        <mechanical_reduction>1.0</mechanical_reduction>
+        </joint>
+    </transmission>
+    <transmission name="back_left_wheel_transmission">
+        <plugin>transmission_interface/SimpleTransmission</plugin>
+        <actuator name="back_wheel_left_motor" role="back_actuator_left"/>
+        <joint name="back_wheel_left_joint"    role="back_joint_left">
+        <mechanical_reduction>1.0</mechanical_reduction>
+        </joint>
+    </transmission>
     <ros2_control name="RobotSystem" type="system">
         <!-- ros2_control Gazebo -->

Commit message: robit_cube_with_motion

File: robitcubebot_description/urdf/lidar.xacro (robot description, xacro)
@@ -2,7 +2,7 @@
 <robot xmlns:xacro="http://www.ros.org/wiki/xacro" >
     <joint name="laser_joint" type="fixed">
-        <parent link="base_link"/>
+        <parent link="upper_link"/>
         <child link="laser_frame"/>
-        <origin xyz="0 -0.005 0.12" rpy="0 0 0"/>
+        <origin xyz="-${base_length /2.5} 0.005 0.06" rpy="0 0 0"/>
     </joint>
     <link name="laser_frame">

File: robitcubebot_description/urdf/robitcubebot_base.xacro (robot description, xacro)
@@ -13,5 +13,5 @@
                            xyz="0 0 ${base_height / 2.0}" rpy="0 0 0" />
     <visual>
-      <origin xyz="${base_length / 2.0} ${base_width / 2.0} 0" rpy="0 0 3.14" />
+      <origin xyz="-${base_length / 2.0} -${base_width / 2.0} 0" rpy="0 0 0" />
       <geometry>
         <mesh filename="package://robitcubebot_description/meshes/base_link.STL" scale="0.001 0.001 0.001" />
@@ -35,5 +35,5 @@
   </joint>
   <!-- Wheels -->
-  <link name="back_wheel_left_link">
+  <link name="front_wheel_right_link">
     <inertial>
       <origin xyz="0 -0.014 0" rpy="0 0 0" />
@@ -56,12 +56,12 @@
     </collision>
   </link>
-  <joint name="back_wheel_left_joint" type="continuous">
-    <origin xyz="-${base_width / 1.8} -${base_width / 2} ${wheel_radius}" rpy="0 0 0" />
+  <joint name="front_wheel_right_joint" type="continuous">
+    <origin xyz="-${base_width / 1.8} -${base_width / 2.1} ${wheel_radius}" rpy="0 0 0" />
     <parent link="base_link" />
-    <child link="back_wheel_left_link" />
-    <axis xyz="0 1 0" />
+    <child link="front_wheel_right_link" />
+    <axis xyz="0 -1 0" />
   </joint>
   <link
-    name="back_wheel_right_link">
+    name="front_wheel_left_link">
     <inertial>
       <origin xyz="0 0.014 0" rpy="0 0 0" />
@@ -84,11 +84,11 @@
     </collision>
   </link>
-  <joint name="back_wheel_right_joint" type="continuous">
+  <joint name="front_wheel_left_joint" type="continuous">
     <origin xyz="-${base_width / 1.8} ${base_width / 2.1} ${wheel_radius}" rpy="0 0 0" />
     <parent link="base_link" />
-    <child link="back_wheel_right_link" />
-    <axis xyz="0 1 0" />
+    <child link="front_wheel_left_link" />
+    <axis xyz="0 -1 0" />
   </joint>
-  <link name="front_wheel_left_link">
+  <link name="back_wheel_right_link">
     <inertial>
       <origin xyz="0 -0.014 0" rpy="0 0 0" />
@@ -111,12 +111,12 @@
     </collision>
   </link>
-  <joint name="front_wheel_left_joint" type="continuous">
-    <origin xyz="${base_width / 1.8} -${base_width / 2} ${wheel_radius}" rpy="0 0 0" />
+  <joint name="back_wheel_right_joint" type="continuous">
+    <origin xyz="${base_width / 1.8} -${base_width / 2.1} ${wheel_radius}" rpy="0 0 0" />
     <parent link="base_link" />
-    <child link="front_wheel_left_link" />
-    <axis xyz="0 1 0" />
+    <child link="back_wheel_right_link" />
+    <axis xyz="0 -1 0" />
   </joint>
   <link
-    name="front_wheel_right_link">
+    name="back_wheel_left_link">
     <inertial>
       <origin xyz="0 0.014 0" rpy="0 0 0" />
@@ -139,9 +139,9 @@
     </collision>
   </link>
-  <joint name="front_wheel_right_joint" type="continuous">
+  <joint name="back_wheel_left_joint" type="continuous">
     <origin xyz="${base_width / 1.8} ${base_width / 2.1} ${wheel_radius}" rpy="0 0 0" />
     <parent link="base_link" />
-    <child link="front_wheel_right_link" />
-    <axis xyz="0 1 0" />
+    <child link="back_wheel_left_link" />
+    <axis xyz="0 -1 0" />
   </joint>
   <link name="upper_link">
@@ -149,5 +149,5 @@
                            xyz="0 0 ${base_height / 2.0}" rpy="0 0 0" />
     <visual>
-      <origin xyz="${base_length / 1.75} 0.165 0" rpy="0 0 3.14" />
+      <origin xyz="-${base_length / 1.75} -0.165 0" rpy="0 0 0" />
       <geometry>
         <mesh filename="package://robitcubebot_description/meshes/upper_link.STL" scale="0.001 0.001 0.001" />

File: robitcubebot_description/urdf/robitcubebot_gazebo.xacro (robot description, xacro)
@@ -9,15 +9,15 @@
     </joint>
   </transmission>
+  <transmission name="back_right_wheel_transmission">
+    <plugin>transmission_interface/SimpleTransmission</plugin>
+    <actuator name="back_wheel_right_motor" role="back_actuator_right"/>
+    <joint name="back_wheel_right_joint"    role="back_joint_right">
+      <mechanical_reduction>1.0</mechanical_reduction>
+    </joint>
+  </transmission>
   <transmission name="front_left_wheel_transmission">
     <plugin>transmission_interface/SimpleTransmission</plugin>
     <actuator name="front_wheel_left_motor" role="front_actuator_left"/>
     <joint name="front_wheel_left_joint"    role="front_joint_left">
-      <mechanical_reduction>1.0</mechanical_reduction>
-    </joint>
-  </transmission>
-  <transmission name="back_right_wheel_transmission">
-    <plugin>transmission_interface/SimpleTransmission</plugin>
-    <actuator name="back_wheel_right_motor" role="back_actuator_right"/>
-    <joint name="back_wheel_right_joint"    role="back_joint_right">
       <mechanical_reduction>1.0</mechanical_reduction>
     </joint>
@@ -31,13 +31,4 @@
   </transmission>
   <!-- Wheels -->
-  <gazebo reference="front_wheel_left_link">
-    <mu1>1000000000000000.0</mu1>
-    <mu2>1000000000000000.0</mu2>
-    <kp>1000000000000.0</kp>
-    <kd>10.0</kd>
-    <minDepth>0.001</minDepth>
-    <maxVel>0.1</maxVel>
-    <fdir1>1 0 0</fdir1>
-  </gazebo>
   <gazebo reference="front_wheel_right_link">
     <mu1>1000000000000000.0</mu1>
@@ -56,4 +47,13 @@
     <minDepth>0.001</minDepth>
     <maxVel>1.0</maxVel>
+  </gazebo>
+  <gazebo reference="front_wheel_left_link">
+    <mu1>1000000000000000.0</mu1>
+    <mu2>1000000000000000.0</mu2>
+    <kp>1000000000000.0</kp>
+    <kd>10.0</kd>
+    <minDepth>0.001</minDepth>
+    <maxVel>0.1</maxVel>
+    <fdir1>1 0 0</fdir1>
   </gazebo>
   <gazebo reference="back_wheel_right_link">

File: robitcubebot_description/urdf/robitcubebot_ros2_control.xacro (robot description, xacro)
@@ -18,6 +18,14 @@
         <joint name="front_wheel_right_joint">
             <command_interface name="velocity">
-              <param name="min">-1</param>
-              <param name="max">1</param>
+              <param name="min">-10</param>
+              <param name="max">10</param>
+            </command_interface>
+            <state_interface name="position" />
+            <state_interface name="velocity" />
+        </joint>
+        <joint name="back_wheel_right_joint">
+            <command_interface name="velocity">
+              <param name="min">-10</param>
+              <param name="max">10</param>
             </command_interface>
             <state_interface name="position" />
@@ -26,14 +34,6 @@
         <joint name="front_wheel_left_joint">
             <command_interface name="velocity">
-              <param name="min">-1</param>
-              <param name="max">1</param>
-            </command_interface>
-            <state_interface name="position" />
-            <state_interface name="velocity" />
-        </joint>
-        <joint name="back_wheel_right_joint">
-            <command_interface name="velocity">
-              <param name="min">-1</param>
-              <param name="max">1</param>
+              <param name="min">-10</param>
+              <param name="max">10</param>
             </command_interface>
             <state_interface name="position" />
@@ -42,6 +42,6 @@
         <joint name="back_wheel_left_joint">
             <command_interface name="velocity">
-              <param name="min">-1</param>
-              <param name="max">1</param>
+              <param name="min">-10</param>
+              <param name="max">10</param>
             </command_interface>
             <state_interface name="position" />

Commit message: lifter_node_unadjusted

File: robitcubebot_description/urdf/lidar.xacro (robot description, xacro)
@@ -4,5 +4,5 @@
         <parent link="base_link"/>
         <child link="laser_frame"/>
-        <origin xyz="0 -0.005 0.12" rpy="0 0 0"/>
+        <origin xyz="0.1 -0.005 0.08" rpy="0 0 0"/>
     </joint>
     <link name="laser_frame">

Commit message: lidar_stl

File: robitcubebot_description/urdf/lidar.xacro (robot description, xacro)
@@ -1,18 +1,40 @@
 <?xml version="1.0"?>
 <robot xmlns:xacro="http://www.ros.org/wiki/xacro" >
-    <joint name="laser_joint" type="fixed">
-        <parent link="base_link"/>
-        <child link="laser_frame"/>
-        <origin xyz="0 -0.005 0.12" rpy="0 0 0"/>
+    <!--link name="laser_frame">
+      <visual>
+        <origin xyz="0 0 0" rpy="0 0 0" />
+        <geometry>
+          <mesh filename="package://robitcubebot_description/meshes/lidar.STL" scale="0.001 0.001 0.001" />
+        </geometry>
+        <material name="black">
+          <color rgba="0.1 0.1 0.1 1" />
+        </material>
+      </visual>
+          <collision>
+              <geometry>
+                  <cylinder radius="0.034" length="0.03"/>
+              </geometry>
+          </collision>
+          <xacro:cylinder_inertia m="1.0" r="${2*0.05}" h="${2*0.04}"
+                                      xyz="0 0 0" rpy="${pi / 2.0} 0 0" />
+    </link-->
+    <joint name="laser_joint_down" type="fixed">
+        <parent link="upper_link"/>
+        <child link="laser_frame_down"/>
+        <origin xyz="0.1  0 0.01" rpy="0 0 0"/>
     </joint>
-    <link name="laser_frame">
+    <link name="laser_frame_down">
         <visual>
+            <origin xyz="0.06  -0.1 -0.043" rpy="1.57 0 3.14"/>
             <geometry>
-                <cylinder radius="0.034" length="0.03"/>
+                <mesh filename="package://robitcubebot_description/meshes/lidar.STL" scale="0.001 0.001 0.001" />
             </geometry>
+            <material name="grey">
+                <color rgba="0.4 0.4 0.4 1" />
+            </material>
         </visual>
         <collision>
             <geometry>
-                <cylinder radius="0.034" length="0.03"/>
+                <mesh filename="package://robitcubebot_description/meshes/lidar.STL" scale="0.001 0.001 0.001" />
             </geometry>
         </collision>
@@ -20,31 +42,3 @@
                                     xyz="0 0 0" rpy="${pi / 2.0} 0 0" />
     </link>
-    <gazebo reference="laser_frame">
-        <material>Gazebo/Red</material>
-        <sensor name="laser" type="ray">
-            <pose> 0 0 0 0 0 0 </pose>
-            <visualize>true</visualize>
-            <update_rate>10</update_rate>
-            <ray>
-                <scan>
-                    <horizontal>
-                        <samples>360</samples>
-                        <min_angle>-3.14</min_angle>
-                        <max_angle>3.14</max_angle>
-                    </horizontal>
-                </scan>
-                <range>
-                    <min>0.3</min>
-                    <max>12</max>
-                </range>
-            </ray>
-            <plugin name="laser_controller" filename="libgazebo_ros_ray_sensor.so">
-                <ros>
-                    <argument>~/out:=scan</argument>
-                </ros>
-                <output_type>sensor_msgs/LaserScan</output_type>
-                <frame_name>laser_frame</frame_name>
-            </plugin>
-        </sensor>
-    </gazebo>
 </robot>
