Commit message: control_plugin_was_Calledtwice

File: robitcubebot_description/urdf/robitcubebot.urdf.xacro (robot description, xacro)
@@ -4,39 +4,6 @@
   <xacro:arg name="is_sim" default="true"/>
   <!-- Include Gazebo Parameters -->
-  <!--xacro:include filename="robitcubebot_gazebo.xacro" /-->
+  <xacro:include filename="robitcubebot_gazebo.xacro" />
   <!-- Move this one to ros2 control -->
-  <transmission name="wheel_right_transmission">
-    <plugin>transmission_interface/SimpleTransmission</plugin>
-    <actuator name="wheel_right_motor" role="actuator_right"/>
-    <joint name="wheel_right_joint"    role="joint_right">
-      <mechanical_reduction>1.0</mechanical_reduction>
-    </joint>
-  </transmission>
-  <transmission name="wheel_left_transmission">
-    <plugin>transmission_interface/SimpleTransmission</plugin>
-    <actuator name="wheel_left_motor" role="actuator_left"/>
-    <joint name="wheel_left_joint"    role="joint_left">
-      <mechanical_reduction>1.0</mechanical_reduction>
-    </joint>
-  </transmission>
-  <!-- Wheels -->
-  <gazebo reference="wheel_left_link">
-    <mu1>1000000000000000.0</mu1>
-    <mu2>1000000000000000.0</mu2>
-    <kp>1000000000000.0</kp>
-    <kd>10.0</kd>
-    <minDepth>0.001</minDepth>
-    <maxVel>0.1</maxVel>
-    <fdir1>1 0 0</fdir1>
-  </gazebo>
-  <gazebo reference="wheel_right_link">
-    <mu1>1000000000000000.0</mu1>
-    <mu2>1000000000000000.0</mu2>
-    <kp>1000000000000.0</kp>
-    <kd>10.0</kd>
-    <minDepth>0.001</minDepth>
-    <maxVel>0.1</maxVel>
-    <fdir1>1 0 0</fdir1>
-  </gazebo>
   <!-- Include ros2_control Plugins -->
   <xacro:include filename="common_properties.xacro" />

File: robitcubebot_description/urdf/robitcubebot_base.xacro (robot description, xacro)
@@ -13,7 +13,5 @@
   <xacro:property name="to_wheel_center" value="0.07" />
   <!-- Include Gazebo Parameters -->
-  <xacro:include filename="$(find robitcubebot_description)/urdf/robitcubebot_gazebo.xacro" />
   <!-- Include ros2_control Plugins -->
-  <xacro:include filename="$(find robitcubebot_description)/urdf/robitcubebot_ros2_control.xacro" />
   <link name="base_footprint"/>
   <link name="base_link">

Commit message: simulation_controller_but_not_completed_hardware

File: robitcubebot_description/urdf/robitcubebot.urdf.xacro (robot description, xacro)
@@ -3,12 +3,18 @@
   <!-- Load Simulated or Real Hardware Interfaces -->
   <xacro:arg name="is_sim" default="true"/>
+  <xacro:arg name="use_ros2_control" default="true"/>
   <!-- Include ros2_control Plugins -->
   <xacro:include filename="common_properties.xacro" />
-  <!--xacro:include filename="$(find robitcubebot_description)/urdf/robitcubebot_ros2_control.xacro" /-->
   <xacro:include filename="robitcubebot_base.xacro" />
   <!-- Include Gazebo Parameters -->
-  <xacro:include filename="robitcubebot_gazebo.xacro" />
-  <xacro:include filename="gazebo_control.xacro" />
+  <!--xacro:include filename="gazebo_control_plugin.xacro" /-->
   <xacro:include filename="lidar.xacro"/>
+  <xacro:if value="$(arg use_ros2_control)">
+      <xacro:include filename="robitcubebot_ros2_control.xacro" />
+      <!--xacro:include filename="robitcubebot_hardware_ros2_control.xacro" /-->
+  </xacro:if>
+  <xacro:unless value="$(arg use_ros2_control)">
+      <xacro:include filename="gazebo_control_plugin.xacro" />
+  </xacro:unless>
   <!--xacro:include filename="lift.xacro" /-->
   <!--xacro:include filename="imu.xacro" /-->

File: robitcubebot_description/urdf/robitcubebot_base.xacro (robot description, xacro)
@@ -40,7 +40,6 @@
             <collision>
                 <geometry>
-                    <cylinder radius="${wheel_radius}" length="${wheel_length}" />
+                    <sphere radius="${wheel_radius}"/>
                 </geometry>
-                <origin xyz="0 0 0" rpy="${pi / 2.0} 0 0" />
             </collision>
             <xacro:cylinder_inertia m="1.0" r="${2*wheel_radius}" h="${2*wheel_length}"

File: robitcubebot_description/urdf/robitcubebot_hardware_ros2_control.xacro (robot description, xacro)
@@ -1,7 +1,14 @@
 <?xml version="1.0"?>
 <robot xmlns:xacro="http://www.ros.org/wiki/xacro" name="robitcubebot">
-    <ros2_control name="GazeboSystem" type="system">
+    <ros2_control name="RealRobot" type="system">
         <hardware>
-            <plugin>gazebo_ros2_control/GazeboSystem</plugin>
+            <plugin>diffdrive_arduino/DiffDriveArduinoHardware</plugin>
+            <param name="left_wheel_name">front_wheel_left_joint</param>
+            <param name="right_wheel_name">front_wheel_right_joint</param>
+            <param name="loop_rate">30</param>
+            <param name="device">/dev/ttyUSB0</param>
+            <param name="baud_rate">57600</param>
+            <param name="timeout">1000</param>
+            <param name="enc_counts_per_rev">3436</param>
         </hardware>
         <joint name="front_wheel_left_joint">
@@ -21,5 +28,5 @@
             <state_interface name="position"/>
         </joint>
-        <joint name="back_wheel_left_joint">
+        <!--joint name="back_wheel_left_joint">
             <command_interface name="velocity">
                 <param name="min">-10</param>
@@ -36,10 +43,5 @@
             <state_interface name="velocity"/>
             <state_interface name="position"/>
-        </joint>
+        </joint-->
     </ros2_control>
-    <gazebo>
-        <plugin name="gazebo_ros2_control" filename="libgazebo_ros2_control.so">
-            <parameters>$(find robitcubebot_bringup)/config/robitcube_controller.yaml</parameters>
-        </plugin>
-    </gazebo>
 </robot>
