Commit message: lift_update

File: robitcubebot_description/urdf/lift.xacro (robot description, xacro)
@@ -6,6 +6,6 @@
   <xacro:property name="screw_length" value="0.10" />
   <link name="link_platform_mid">
-    <origin xyz="0 0 0.0" rpy="0 0 0"/>
     <visual>
+      <origin xyz="0 0 0.045" rpy="0 0 0"/>
       <geometry>
         <mesh filename="package://robitcubebot_description/meshes/Lead_screw.STL" scale="0.001 0.001 0.001" />
@@ -14,10 +14,5 @@
           <color rgba="0.1 0.1 0.1 1" />
       </material>
-    </visual>
-    <collision>
-      <geometry>
-        <box size="0.02 0.02 0.10" />
-      </geometry>
-    </collision>
+      </visual>
     <inertial>
       <mass value="1"/>
@@ -57,5 +52,5 @@
   </link>
   <joint name="lift_joint" type="prismatic" >
-    <origin xyz="0 0 0.08" rpy="0 0 0"/>
+    <origin xyz="0 0 0.1" rpy="0 0 0"/>
     <child link="lift_link" />
     <parent link="link_platform_mid" />

Commit message: diffdrive_plugin_with_lifter

File: robitcubebot_description/urdf/lift.xacro (robot description, xacro)
@@ -5,37 +5,19 @@
   <xacro:property name="plate_radius" value="0.045" />
   <xacro:property name="screw_length" value="0.10" />
+  <xacro:macro name="lifter_transmission" params="joint_name actuator_name">
+    <transmission name="${joint_name}_transmission">
+        <plugin>transmission_interface/SimpleTransmission</plugin>
+        <actuator name="${actuator_name}" role="actuator1"/>
+        <joint name="${joint_name}" role="joint1">
+            <mechanical_reduction>1.0</mechanical_reduction>
+        </joint>
+    </transmission>
+  </xacro:macro>
+   <!-- Link for the platform mid -->
   <link name="link_platform_mid">
     <origin xyz="0 0 0.0" rpy="0 0 0"/>
     <visual>
       <geometry>
-        <mesh filename="package://robitcubebot_description/meshes/Lead_screw.STL" scale="0.001 0.001 0.001" />
-      </geometry>
-      <material name="black">
-          <color rgba="0.1 0.1 0.1 1" />
-      </material>
-    </visual>
-    <collision>
-      <geometry>
-        <box size="0.02 0.02 0.10" />
-      </geometry>
-    </collision>
-    <inertial>
-      <mass value="1"/>
-      <inertia
-              ixx="1.0" ixy="0.0" ixz="0.0"
-              iyy="1.0" iyz="0.0"
-              izz="1.0"/>
-    </inertial>
-  </link>
-  <joint name="platform_joint" type="fixed">
-    <parent link="base_link" />
-    <child link="link_platform_mid" />
-    <origin xyz="0.0 0 ${robot_height}" rpy="0. 0. 0."/>
-  </joint>
-  <link name="lift_link">
-    <visual>
-      <origin xyz="-${plate_radius/1.1} -${plate_radius/1.1}  0.0" rpy="0 0 0"/>
-      <geometry>
-        <mesh filename="package://robitcubebot_description/meshes/upperstand.STL" scale="0.001 0.001 0.001" />
+        <cylinder radius="0.005" length="0.04"/>
       </geometry>
       <material name="black">
@@ -45,22 +27,42 @@
     <collision>
       <geometry>
-         <mesh filename="package://robitcubebot_description/meshes/upperstand.STL" scale="0.001 0.001 0.001" />
+         <cylinder radius="0.01" length="0.04"/>
       </geometry>
     </collision>
     <inertial>
       <mass value="1"/>
-      <inertia
-              ixx="1.0" ixy="0.0" ixz="0.0"
-              iyy="1.0" iyz="0.0"
-              izz="1.0"/>
+      <inertia ixx="1.0" ixy="0.0" ixz="0.0"
+               iyy="1.0" iyz="0.0"
+               izz="1.0"/>
     </inertial>
   </link>
-  <joint name="lift_joint" type="prismatic">
-    <origin xyz="0 0 0.03" rpy="0 0 0"/>
-    <parent link="link_platform_mid" />
-    <child link="lift_link" />
-    <axis xyz="0 0 1" rpy="0 0 0"/>
-    <limit effort="100.0" lower="-0.05" upper="0.035" velocity="1.0"/>
-    <dynamics damping="0.1" friction="0.1"/>
+  <!-- Joint connecting upper link to platform mid -->
+  <joint name="platform_joint" type="fixed">
+    <parent link="base_link" />
+    <child link="link_platform_mid" />
+    <origin xyz="0.0 0 ${robot_height+0.015}" rpy="0 0 0"/>
   </joint>
+  <!-- Link for the lift mechanism -->
+  <link name="lift_link">
+    <visual>
+      <origin xyz="0 0  0.0" rpy="0 0 0"/>
+      <geometry>
+        <cylinder radius="0.06" length="0.0015"/>
+      </geometry>
+      <material name="black">
+        <color rgba="0.1 0.1 0.1 1" />
+      </material>
+    </visual>
+    <collision>
+      <geometry>
+        <cylinder radius="0.08" length="0.001"/>
+      </geometry>
+    </collision>
+    <inertial>
+      <mass value="1"/>
+      <inertia ixx="1.0" ixy="0.0" ixz="0.0"
+               iyy="1.0" iyz="0.0"
+               izz="1.0"/>
+    </inertial>
+  </link>
 </robot>

File: robitcubebot_description/urdf/robitcubebot.urdf.xacro (robot description, xacro)
@@ -3,5 +3,5 @@
   <!-- Load Simulated or Real Hardware Interfaces -->
   <xacro:arg name="is_sim" default="true"/>
-  <xacro:arg name="use_ros2_control" default="true"/>
+  <xacro:arg name="use_ros2_control" default="false"/>
   <!-- Include ros2_control Plugins -->
   <xacro:include filename="common_properties.xacro" />
@@ -17,5 +17,6 @@
       <xacro:include filename="gazebo_control_plugin.xacro" />
   </xacro:unless>
-  <!--xacro:include filename="lift.xacro" /-->
+  <xacro:include filename="lift.xacro" />
+  <xacro:include filename="lift_controller.xacro" />
   <!--xacro:include filename="imu.xacro" /-->
 </robot>

Commit message: updating lift limits, adding moviet script

File: robitcubebot_description/urdf/lift.xacro (robot description, xacro)
@@ -48,5 +48,5 @@
       <origin xyz="0 0  0.0" rpy="0 0 0"/>
       <geometry>
-        <cylinder radius="0.06" length="0.0015"/>
+        <cylinder radius="0.09" length="0.0015"/>
       </geometry>
       <material name="black">
@@ -56,6 +56,27 @@
     <collision>
       <geometry>
-        <cylinder radius="0.08" length="0.001"/>
+        <cylinder radius="0.1" length="0.001"/>
       </geometry>
+      <surface>
+        <friction>
+          <ode>
+            <mu>1.0</mu>
+            <mu2>1.0</mu2>
+          </ode>
+          <torsional>
+            <ode>
+              <slip>0.0</slip>
+            </ode>
+          </torsional>
+        </friction>
+        <contact>
+          <ode>
+            <soft_cfm>0.0</soft_cfm>
+            <soft_erp>0.2</soft_erp>
+            <kp>100000.0</kp>
+            <kd>1.0</kd>
+          </ode>
+        </contact>
+      </surface>
     </collision>
     <inertial>

File: robitcubebot_description/urdf/lift_controller.xacro (robot description, xacro)
@@ -8,5 +8,5 @@
       <joint name="lift_joint">
           <command_interface name="position">
-          <param name="min">-05</param>
+          <param name="min">-0.035</param>
           <param name="max">1.5</param>
           </command_interface>
@@ -20,5 +20,5 @@
     <child link="lift_link" />
     <axis xyz="0 0 1" rpy="0 0 0"/>
-    <limit effort="100.0" lower="-0.035" upper="-0.015" velocity="1.0"/>
+    <limit effort="10000.0" lower="-0.035" upper="1.0" velocity="1.0"/>
     <dynamics damping="0.1" friction="0.1"/>
     <hardwareInterface>hardware_interface/VelocityJointInterface</hardwareInterface>
